File: AutoSteer6 PCB/AutoSteer6.sch (KiCad schematic (older format))
At the start: 40 parts, among them J1 SDA, J10 Roll/Pitch, J11 Power In, J2 SCL, J3 I2C-1, J4 I2C-1, J5 Steering, J6 Power Source, J7 VCC, J8 Motor Control, J9 Motor Power, U1 ADS1115

Commit message: minor changes
Parts:
- removed C13: 0.1 uF, Capacitor_THT:C_Disc_D5.0mm_W2.5mm_P2.50mm, symbol Device:CP
- removed J3: I2C-1, Connector_PinHeader_2.54mm:PinHeader_1x04_P2.54mm_Vertical, symbol Connector:Conn_01x04_Female
- removed R1: 330, Resistor_THT:R_Axial_DIN0204_L3.6mm_D1.6mm_P7.62mm_Horizontal, symbol Device:R
- J3: renamed from J4; value I2C-1 -> I2C-5V
- renumbered C2 to C1, C14 to C10, C8 to C11, C10 to C12, C11 to C13, C15 to C14, C16 to C15, C1 to C2, C12 to C8, D2 to D1, D1 to D2, J11 to J10, J5 to J4, J6 to J5, J7 to J6, J10 to J7, R7 to R1, R3 to R2, R2 to R3
Connections:
- net at C7.1, R2.1: now also A1.22 (D4); no longer A1.21 (D3)
- net at A1.25 (D7): now also C9.1, R3.1
- net at A1.26 (D8): now also C10.1, J8.1 (Pin_1)
- net at A1.27 (D9), C11.1: now also J8.2 (Pin_2); no longer J8.1 (Pin_1)
- net at A1.28 (D10): no longer J8.2 (Pin_2)
- net at A1.30 (D12): no longer C9.1
- net at C1.1, C14.1, C2.1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: now also J4.1 (Pin_1), R1.1; no longer R1.2
- net at D1.2 (A): now also R1.2; no longer R1.1
- now unconnected: A1.29 (D11)
- no-connect marks 21 -> 22
Other:
- moved on the sheet: C10, C11, C15, C7, C8, D1, D2, J10, J3, J7, R1, R2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

Commit message: update pcb
Parts:
- removed C10, C11, C12, C13, C5, C6, C7, C8, C9: 0.1 uF, Capacitor_THT:C_Disc_D5.0mm_W2.5mm_P2.50mm, symbol Device:CP
- removed J4: Steering, my library:Phoenix_16_pin_5mm_terminal_block, symbol Connector:Screw_Terminal_01x16
- removed J7: Roll/Pitch, my library:Phoenix_4_pin_5mm_terminal_block, symbol Connector:Screw_Terminal_01x04
- removed J8: Motor Control, my library:Phoenix_3_pin_5mm_terminal_block, symbol Connector:Screw_Terminal_01x03
- removed J9: Motor Power, my library:Phoenix_2_pin_5mm_terminal_block, symbol Connector:Screw_Terminal_01x02
- added J3: Analog, my library:Phoenix_4_pin_5mm_terminal_block, symbol Connector:Screw_Terminal_01x04
- added J5: GPIO's, my library:Phoenix_7_pin_5mm_terminal_block, symbol Connector:Screw_Terminal_01x07
- added J6: Ground, my library:Phoenix_9_pin_5mm_terminal_block, symbol Connector:Screw_Terminal_01x09
- added J8: Power Out, my library:Phoenix_6_pin_5mm_terminal_block, symbol Connector:Screw_Terminal_01x06
- renumbered C14 to C5, C15 to C6, J6 to J10, J3 to J4, J5 to J7, J10 to J9, R4 to R2, R2 to R3, R3 to R4, R6 to R5, R5 to R6
Connections:
- net GND: now also J9.1 (Pin_1), J6.1 (Pin_1), J6.2 (Pin_2), J6.3 (Pin_3), J6.4 (Pin_4), J6.5 (Pin_5), J6.6 (Pin_6), J6.7 (Pin_7), J6.8 (Pin_8), J6.9 (Pin_9); no longer J9.2 (Pin_2)
- net at A1.20 (D2): now also R2.2; no longer R2.1
- net at A1.22 (D4): now also R3.2; no longer R3.1
- net at A1.23 (D5): now also J5.3 (Pin_3)
- net at A1.24 (D6): now also J5.4 (Pin_4)
- net at A1.25 (D7): now also R4.2; no longer R4.1
- net at A1.26 (D8): now also J5.6 (Pin_6)
- net at A1.27 (D9): now also J5.7 (Pin_7)
- net at C1.1, C2.1, C3.1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: now also J8.4 (Pin_4), J8.5 (Pin_5)
- net at U1.10 (AIN3): now also J3.1 (Pin_1)
- net at J2.3 (Pin_3), J4.3 (Pin_3), U1.3 (SCL): now also L1.7 (HV1); no longer L1.12 (HV4)
- net at J1.3 (Pin_3), J4.4 (Pin_4), U1.4 (SDA): now also L1.8 (HV2); no longer L1.7 (HV1)
- net at U1.7 (AIN0): now also J3.4 (Pin_4)
- net at U1.8 (AIN1): now also J3.3 (Pin_3)
- net at U1.9 (AIN2): now also J3.2 (Pin_2)
- net at C4.1, C6.1, D2.C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: now also J8.1 (Pin_1), J8.2 (Pin_2), J8.3 (Pin_3)
- net at D2.A: now also J9.2 (Pin_2); no longer J9.1 (Pin_1)
- net at J10.2 (Pin_2), R5.1, R6.1: now also J8.6 (Pin_6)
- net at L1.1 (LV1): now also J2.1 (Pin_1); no longer J1.1 (Pin_1)
- net at L1.2 (LV2): now also J1.1 (Pin_1)
- net at L1.6 (LV4): no longer J2.1 (Pin_1)
- new net: J5.2 (Pin_2), R3.1
- new net: J5.1 (Pin_1), R2.1
- new net: J5.5 (Pin_5), R4.1
- no-connect marks 22 -> 21
Other:
- moved on the sheet: A1, C1, C2, C3, C4, C5, C6, D1, D2, J1, J10, J2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
