File: PCBs/AutoSteer12_PCB/TestDesign/AS12.sch (KiCad schematic (older format))
At the start: 66 parts, among them IC1 PCA9306DCUR, IC2 LM2576HVR-5.0, J1 ADS1115, J10 Conn_01x08_Female, J11 Teensy_Ethernet, J12 HR911105A, J13 Conn_01x15_Female, J14 Conn_01x08_Female, J15 Motor 2, J16 Motor 1, J17 SF_F9P_left, J18 ArduSimple_tl, J19 ArduSimple_bl, J2 WemosD1_left, J20 SF_F9P_right, J21 ArduSimple_tr, J22 ArduSimple_br, J23 Grove, J24 WemosD1_right, J3 DT13-12PA, J4 CMPS14, J5 BNO080_left, J6 BNO080_right, J7 I2C-3V3, J8 I2C-3V3, J9 Conn_01x15_Female, K1 HF3FF_012-1ZST, Q1 BC847, U1 PC817X2CSP9F, U2 PC817X2CSP9F, U3 PC817X2CSP9F, U4 CC6900SO-10A, U5 AZ1117H-3.3TRE1, U6 MAX3485EESA+T, U7 PC817X2CSP9F

Commit message: update pcb/software
Parts:
- removed IC2: LM2576HVR-5.0, MyFootprints:TO263-5L, symbol AS12-rescue:LM2576HV_TO-263-5L-MyLib
- removed U5: AZ1117H-3.3TRE1, Package_TO_SOT_SMD:SOT-223, symbol AS12-rescue:AZ1117H-3.3TRE1-MyLib
- added C2: CL21B105KAFNNNE, Capacitor_SMD:C_0805_2012Metric, symbol Device:C
- added D5, D6: Zener Diode, Diode_SMD:D_SOD-123F, symbol Device:D_Zener
- added IC2: XL2596, MyFootprints:TO263-5L, symbol MyLib:XL2596
- added IC3: AZ1117, Package_TO_SOT_SMD:SOT-223, symbol MyLib:AZ1117
- added KF2: KF142V-5.0-2P, MyFootprints:KF142V-5.08-2P, symbol MyLib:KF142V-5.0-2P
- added R13, R14: 200, Resistor_SMD:R_1210_3225Metric, symbol Device:R
- C10: value VEJ102M1ETR-1313 -> RVT1V331M1010; footprint MyFootprints:CAPAE1300X1400N -> Capacitor_SMD:CP_Elec_10x10.5
- C9: value RVT1J101M1010 -> RVT1V471M1010; footprint Capacitor_SMD:CP_Elec_10x10 -> Capacitor_SMD:CP_Elec_10x10.5
- D4: footprint MyFootprints:1N4007 -> Diode_SMD:D_SMA
- L1: value TMPA1265SP-101MN-D -> SMDRI127-330MT
Connections:
- net GND: now also C2.2, D5.2 (A), D6.2 (A), IC2.3 (GND), IC2.5 (On/Off), IC2.6 (GND_1), IC3.1 (ADJ/GND)
- net at C10.1, C11.1, C12.1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: now also IC2.4 (Feedback), IC3.3 (INPUT)
- net at C1.1, C4.1, C5.1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: now also IC3.2 (OUTPUT)
- net at J10.1 (Pin_1): now also R13.2
- net at J10.2 (Pin_2): now also R14.2; no longer U3.4
- net at J14.3 (Pin_3): now also U3.4
- net at D2.1, L1.1: now also IC2.2 (Output)
- net at C9.1, D3.1 (K): now also C2.1, IC2.1 (VIN)
- new net: D6.1 (K), KF2.1, R13.1
- new net: D5.1 (K), KF2.2, R14.1
Other:
- moved on the sheet: C6, C7, C9, D1, D2, D3, F1, R4, R5

Commit message: fix board errors
Parts:
- removed C6: 10uF, Capacitor_SMD:C_0805_2012Metric, symbol Device:CP
- removed D2: SS36, DIOM8059X265N, symbol SamacSys_Parts:SS36
- added C6: 10uF, Capacitor_SMD:C_0805_2012Metric, symbol Device:C
- added D2: D_Schottky, MyFootprints:SMA(DO-214AC), symbol Device:D_Schottky
- added J25: RS485, MyFootprints:Qwic_vertical, symbol Connector_Generic:Conn_01x04
- IC1: symbol AS12-rescue:PCA9306DCUR-SamacSys_Parts -> SamacSys_Parts:PCA9306DCUR
- J12: symbol AS12-rescue:HR911105A-MyLib -> MyLib:HR911105A
- J23: symbol AS12-rescue:Grove-MyLib -> MyLib:Grove
- J3: symbol AS12-rescue:DT13-12PA-MyLib -> MyLib:DT13-12PA
- K1: symbol AS12-rescue:HF3FF_012-1ZST-HF3FF_012-1ZST -> MyLib:HF3FF_012-1ZST
- KF1: symbol AS12-rescue:KF142V-5.0-6P-MyLib -> MyLib:KF142V-5.0-6P
- U4: symbol AS12-rescue:CH70120CB3PR-MyLib -> MyLib:CH70120CB3PR
- U6: footprint MyFootprints:MAX485ESA&plus_T -> MyFootprints:Maxim_Integrated-S8-2-0-P-MFG
Connections:
- wire segments 403 -> 411
Other:
- note added: "12V"
- note added: "25"
- note added: "26"
- note removed: "12V In"
- moved on the sheet: F1
