File: PCBs/AutoSteer13-2_PCB/AS13.kicad_pcb (KiCad board)
At the start: 2 copper layers, 159 x 159 mm, 86 parts, among them IC1 AZ1117, IC2 XL2596, J1 U-USBAS04P-F000, J10 I2C-3V3, J11 I2C-3V3, J12 CMPS14, J13 Conn_01x15_Female, J14 Conn_01x08_Female, J15 BNO080_left, J16 BNO080_right, J17 Conn_01x15_Female, J18 Conn_01x08_Female, J19 Motor 2, J2 RS485, J20 Motor 1, J21 SF_F9P_left, J22 ArduSimple_tl, J23 ArduSimple_bl, J24 SF_F9P_right, J25 ArduSimple_tr, J26 ArduSimple_br, J27 Grove, J3 Teensy_USBhost, J4 HR911105A, J5 PM254V-11-06-H85, J6 DT13-12PA, J7 WemosD1_left, J8 Teensy_Ethernet, J9 WemosD1_right, K1 SRD-05VDC-SL-C, Q1 BC847, U1 SP3485EN-L/TR, U2 PC817X2CSP9F, U3 PC817X2CSP9F, U4 PC817X2CSP9F, U5 PC817X2CSP9F, U6 CC6900SO-10A

Commit message: update pcb
Parts:
- removed J12: CMPS14, Connector_PinSocket_2.54mm:PinSocket_1x06_P2.54mm_Vertical
- added D6: MMSZ5231B, Diode_SMD:D_SOD-123F, F.Cu at (128.0, 140.3)
- added M1: CMPS14, MyFootprints:CMPS14_no_pins, F.Cu at (123.9, 111.0)
- added R13: 200, Resistor_SMD:R_1206_3216Metric, F.Cu at (128.1, 144.2)
- added R14: 400, Resistor_SMD:R_1206_3216Metric, F.Cu at (128.0, 136.6)
- moved C10 16.6 mm to (116.1, 126.4), turned to 90 degrees
- moved C4 7.17 mm to (135.9, 146.7), turned to 0 degrees
Connections:
- C4 pad 1: Net-(C1-Pad1) -> Net-(C11-Pad1)
- J13 pad 12: Net-(J13-Pad12) -> Net-(D6-Pad1)
- U6 pad 7: Net-(J13-Pad12) -> Net-(R13-Pad2)
- U6 pad 8: Net-(C1-Pad1) -> Net-(C11-Pad1)
Routing:
- net Net-(J13-Pad12): track 56.0 -> 0.00 mm, vias 1 -> 0
- net Net-(D6-Pad1): track 0.00 -> 51.6 mm, vias 0 -> 1
- net Net-(C11-Pad1): track 361.4 -> 382.7 mm
- net Net-(J10-Pad3): track 88.7 -> 69.7 mm
- net Net-(C1-Pad1): track 147.1 -> 128.4 mm
- net Net-(J10-Pad4): track 85.3 -> 69.8 mm
- net Net-(R13-Pad2): track 0.00 -> 5.50 mm
- net GND: track 121.8 -> 127.0 mm, vias 28 -> 30
- net Net-(D2-Pad1): track 65.0 -> 67.5 mm
Other:
- board text added: "AS13 13-Mar-2022"
- board text removed: "AS13 22-Feb-2022"
- board text removed: "CMPS14"
- board text removed: "Factory Use"
- board text removed: "Mode"

Commit message: added BAV99 to analog pins
Parts:
- D1, D2, D6: value MMSZ5231B -> BAV99; footprint Diode_SMD:D_SOD-123F -> Package_TO_SOT_SMD:SOT-23
- R12: footprint Resistor_SMD:R_1210_3225Metric -> Resistor_SMD:R_1206_3216Metric
- R13, R6, R8: value 200 -> 1K
- R14, R7, R9: value 400 -> 2K
- moved D2 38.7 mm to (157.8, 111.3)
- moved D1 37.6 mm to (128.0, 136.2)
- moved R14 17.8 mm to (142.1, 147.3), turned to 0 degrees
- moved R8 16.2 mm to (127.9, 144.3)
- moved R13 15.7 mm to (142.1, 151.1)
- moved R9 14.9 mm to (128.0, 140.6), turned to 0 degrees
- moved D6 14.1 mm to (141.9, 142.8), turned to 180 degrees
- moved R7 5.20 mm to (157.9, 115.8)
- moved R12 1.72 mm to (97.6, 121.7)
- moved R6 1.02 mm to (158.0, 119.6)
- moved C1 0.89 mm to (158.0, 125.2), turned to 270 degrees
Connections:
- D1 pad 1: Net-(D1-Pad1) -> GND
- D1 pad 2: GND -> Net-(C1-Pad1)
- D2 pad 1: Net-(D2-Pad1) -> GND
- D2 pad 2: GND -> Net-(C1-Pad1)
- D6 pad 1: Net-(D6-Pad1) -> GND
- D6 pad 2: GND -> Net-(C1-Pad1)
- J13 pad 12: Net-(D6-Pad1) -> Net-(D1-Pad3)
- J14 pad 1: Net-(D2-Pad1) -> Net-(D6-Pad3)
- J14 pad 2: Net-(D1-Pad1) -> Net-(D2-Pad3)
- J4 pad MH1: (no net) -> GND
- J4 pad MH2: (no net) -> GND
- R13 pad 1: Net-(D6-Pad1) -> Net-(D6-Pad3)
- R13 pad 2: Net-(R13-Pad2) -> Net-(J6-Pad4)
- R14 pad 1: GND -> Net-(D6-Pad3)
- R14 pad 2: Net-(D6-Pad1) -> GND
- R6 pad 1: Net-(D1-Pad1) -> Net-(D2-Pad3)
- R7 pad 1: Net-(D1-Pad1) -> Net-(D2-Pad3)
- R8 pad 1: Net-(J6-Pad4) -> Net-(D1-Pad3)
- R8 pad 2: Net-(D2-Pad1) -> Net-(R8-Pad2)
- R9 pad 1: GND -> Net-(D1-Pad3)
- R9 pad 2: Net-(D2-Pad1) -> GND
- U6 pad 7: Net-(R13-Pad2) -> Net-(R8-Pad2)
Routing:
- net Net-(D2-Pad1): track 67.5 -> 0.00 mm
- net Net-(D6-Pad3): track 0.00 -> 66.3 mm
- net Net-(D6-Pad1): track 51.6 -> 0.00 mm, vias 1 -> 0
- net Net-(D1-Pad3): track 0.00 -> 50.8 mm, vias 0 -> 1
- net Net-(C1-Pad1): track 128.4 -> 162.2 mm, vias 2 -> 4
- net Net-(D2-Pad3): track 0.00 -> 27.1 mm
- net Net-(D1-Pad1): track 24.2 -> 0.00 mm
- net Net-(R13-Pad2): track 5.50 -> 0.00 mm
- net Net-(R8-Pad2): track 0.00 -> 5.38 mm
- net Net-(J14-Pad3): track 33.4 -> 29.8 mm
- net GND: track 127.0 -> 124.0 mm, vias 30 -> 31
- net Net-(J14-Pad4): track 29.9 -> 27.9 mm
- net Net-(J14-Pad5): track 33.8 -> 31.7 mm
- net Net-(KF3-Pad4): track 26.5 -> 25.4 mm
- net Net-(J6-Pad4): track 6.95 -> 5.98 mm
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Other:
- board text added: "AS13-2 14-Mar-2022"
- board text removed: "AS13 13-Mar-2022"
