File: PCBs/AutoSteer13-2_PCB/AS13.sch (KiCad schematic (older format))
At the start: 71 parts, among them IC1 AZ1117, IC2 XL2596, J1 U-USBAS04P-F000, J10 I2C-3V3, J11 I2C-3V3, J12 CMPS14, J13 Conn_01x15_Female, J14 Conn_01x08_Female, J15 BNO080_left, J16 BNO080_right, J17 Conn_01x15_Female, J18 Conn_01x08_Female, J19 Motor 2, J2 RS485, J20 Motor 1, J21 SF_F9P_left, J22 ArduSimple_tl, J23 ArduSimple_bl, J24 SF_F9P_right, J25 ArduSimple_tr, J26 ArduSimple_br, J27 Grove, J3 Teensy_USBhost, J4 HR911105A, J5 PM254V-11-06-H85, J6 DT13-12PA, J7 WemosD1_left, J8 Teensy_Ethernet, J9 WemosD1_right, K1 SRD-05VDC-SL-C, Q1 BC847, U1 SP3485EN-L/TR, U2 PC817X2CSP9F, U3 PC817X2CSP9F, U4 PC817X2CSP9F, U5 PC817X2CSP9F, U6 CC6900SO-10A

Commit message: update pcb
Parts:
- removed J12: CMPS14, Connector_PinSocket_2.54mm:PinSocket_1x06_P2.54mm_Vertical, symbol Connector:Conn_01x06_Female
- added D6: MMSZ5231B, Diode_SMD:D_SOD-123F, symbol Device:D_Zener
- added R13: 200, Resistor_SMD:R_1206_3216Metric, symbol Device:R
- added R14: 400, Resistor_SMD:R_1206_3216Metric, symbol Device:R
Connections:
- net GND: now also D6.2 (A), R14.1
- net at U6.7 (VIOUT): now also R13.2; no longer J13.12 (Pin_12)
- net at C1.1, C10.1, C5.1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: no longer C4.1, U6.8 (VCC)
- net at C11.1, C12.1, C13.1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: now also C4.1, U6.8 (VCC)
- new net: D6.1 (K), J13.12 (Pin_12), R13.1, R14.2
- no-connect marks 87 -> 85
Other:
- moved on the sheet: C4, U6
Changed lines of the file:
@@
 encoding utf-8
 Sheet 1 1
-Title "AS13"
-Date "2022-02-22"
+Title "AS13-2"
+Date "2022-03-13"
 Rev ""
 Comp ""
@@
 L power:GND #PWR017
 U 1 1 61D3D2DF
-P 4450 6600
-F 0 "#PWR017" H 4450 6350 50  0001 C CNN
-F 1 "GND" H 4350 6500 50  0000 C CNN
-F 2 "" H 4450 6600 50  0001 C CNN
-F 3 "" H 4450 6600 50  0001 C CNN
-	1    4450 6600
+P 3500 6650
+F 0 "#PWR017" H 3500 6400 50  0001 C CNN
+F 1 "GND" H 3400 6550 50  0000 C CNN
+F 2 "" H 3500 6650 50  0001 C CNN
+F 3 "" H 3500 6650 50  0001 C CNN
+	1    3500 6650
 	1    0    0    -1
 $EndComp
@@
 Wire Wire Line
 	7400 4600 7400 4050
-Wire Wire Line
-	7400 4050 5900 4050
 Connection ~ 7400 4600
 Connection ~ 5400 4050
@@
 	5550 2550 5550 5550
 Wire Wire Line
-	6000 4900 5800 4900
-Connection ~ 6000 4900
-Wire Wire Line
-	5950 5000 5800 5000
-Connection ~ 5950 5000
-Wire Wire Line
 	5450 3350 5450 4750
 $Comp
-L power:GND #PWR028
-U 1 1 6207AE22
-P 6000 5250
-F 0 "#PWR028" H 6000 5000 50  0001 C CNN
-F 1 "GND" H 6100 5150 50  0000 C CNN
-F 2 "" H 6000 5250 50  0001 C CNN
-F 3 "" H 6000 5250 50  0001 C CNN
-	1    6000 5250
-	1    0    0    -1
-$EndComp
-Wire Wire Line
-	5800 5300 5900 5300
-Wire Wire Line
-	5900 5300 5900 5250
-Wire Wire Line
-	5900 5250 6000 5250
-NoConn ~ 5800 5200
-NoConn ~ 5800 5100
-Wire Wire Line
-	5800 4800 5900 4800
-Wire Wire Line
-	5900 4800 5900 4050
-Connection ~ 5900 4050
-Wire Wire Line
-	5400 4050 5900 4050
-$Comp
 L power:GND #PWR01
 U 1 1 62052DEB
@@
 Wire Wire Line
 	6400 6700 6400 6500
-NoConn ~ 4300 6950
+NoConn ~ 3300 6950
 NoConn ~ 7800 3050
 Wire Wire Line
@@
 	8900 6400 8550 6400
 Wire Wire Line
-	8550 6400 8550 7450
+	8550 6400 8550 7350
 Wire Wire Line
 	8750 6700 8900 6700
@@
 $EndComp
 $Comp
-L Connector:Conn_01x06_Female J12
-U 1 1 61F24CA0
-P 5600 5000
-F 0 "J12" H 5450 5450 50  0000 L CNN
-F 1 "CMPS14" H 5300 5350 50  0000 L CNN
-F 2 "Connector_PinSocket_2.54mm:PinSocket_1x06_P2.54mm_Vertical" H 5600 5000 50  0001 C CNN
-F 3 "~" H 5600 5000 50  0001 C CNN
-	1    5600 5000
-	-1   0    0    -1
-$EndComp
-$Comp
 L MyLib:KF142V-5.0-2P KF1
 U 1 1 61EBE94F
@@
 L Device:CP C4
 U 1 1 61D211FD
-P 4450 6450
-F 0 "C4" H 4200 6450 50  0000 L CNN
-F 1 "0.1uF" H 4200 6350 50  0000 L CNN
-F 2 "Capacitor_SMD:C_0805_2012Metric" H 4488 6300 50  0001 C CNN
-F 3 "~" H 4450 6450 50  0001 C CNN
-	1    4450 6450
+P 3500 6500
+F 0 "C4" H 3250 6500 50  0000 L CNN
+F 1 "0.1uF" H 3250 6400 50  0000 L CNN
+F 2 "Capacitor_SMD:C_0805_2012Metric" H 3538 6350 50  0001 C CNN
+F 3 "~" H 3500 6500 50  0001 C CNN
+	1    3500 6500
 	1    0    0    -1
 $EndComp
@@
 L MyLib:CH70120CB3PR U6
 U 1 1 61C4A961
-P 3900 6850
-F 0 "U6" H 3650 6500 50  0000 C CNN
-F 1 "CC6900SO-10A" H 4200 6500 50  0000 C CNN
-F 2 "MyFootprints:SOIC127P600X175-8N" H 4000 6500 50  0001 L CIN
-F 3 "" H 3900 6850 50  0001 C CNN
-	1    3900 6850
+P 2900 6850
+F 0 "U6" H 2650 6500 50  0000 C CNN
+F 1 "CC6900SO-10A" H 3200 6500 50  0000 C CNN
+F 2 "MyFootprints:SOIC127P600X175-8N" H 3000 6500 50  0001 L CIN
+F 3 "" H 2900 6850 50  0001 C CNN
+	1    2900 6850
 	1    0    0    -1
 $EndComp
-Connection ~ 3450 6750
 Wire Wire Line
-	3450 6650 3500 6650
+	2450 6650 2500 6650
 Wire Wire Line
-	3450 6750 3450 6650
+	2450 6750 2450 6650
 Wire Wire Line
-	3500 6750 3450 6750
+	2500 6750 2450 6750
 Wire Wire Line
-	3500 7050 3500 6950
+	2500 7050 2500 6950
 $Comp
 L power:GND #PWR049
 U 1 1 62313C39
-P 4500 7250
-F 0 "#PWR049" H 4500 7000 50  0001 C CNN
-F 1 "GND" H 4400 7150 50  0000 C CNN
-F 2 "" H 4500 7250 50  0001 C CNN
-F 3 "" H 4500 7250 50  0001 C CNN
-	1    4500 7250
+P 2900 7250
+F 0 "#PWR049" H 2900 7000 50  0001 C CNN
+F 1 "GND" H 2800 7150 50  0000 C CNN
+F 2 "" H 2900 7250 50  0001 C CNN
+F 3 "" H 2900 7250 50  0001 C CNN
+	1    2900 7250
 	1    0    0    -1
 $EndComp
 Wire Wire Line
-	4500 6900 4500 7250
-Wire Wire Line
-	3900 7250 4500 7250
-Connection ~ 4500 7250
-Wire Wire Line
-	4300 6850 4550 6850
-Wire Wire Line
 	4550 5550 4550 6850
 Wire Wire Line
@@
 	4450 5500 5400 5500
 Wire Wire Line
-	4450 6300 3900 6300
-Connection ~ 4450 6300
-Wire Wire Line
 	3700 5450 4250 5450
-Wire Wire Line
-	2350 6950 3500 6950
-Connection ~ 3500 6950
 Connection ~ 6300 5400
 $Comp
 L power:GND #PWR048
 U 1 1 62502EA0
-P 4250 5550
-F 0 "#PWR048" H 4250 5300 50  0001 C CNN
-F 1 "GND" H 4150 5450 50  0000 C CNN
-F 2 "" H 4250 5550 50  0001 C CNN
-F 3 "" H 4250 5550 50  0001 C CNN
-	1    4250 5550
-	1    0    0    -1
+P 3950 5550
+F 0 "#PWR048" H 3950 5300 50  0001 C CNN
+F 1 "GND" V 4000 5400 50  0000 C CNN
+F 2 "" H 3950 5550 50  0001 C CNN
+F 3 "" H 3950 5550 50  0001 C CNN
+	1    3950 5550
+	0    -1   -1   0
 $EndComp
 Wire Wire Line
-	3700 5550 4250 5550
-Wire Wire Line
 	1450 3450 2350 3450
 Wire Wire Line
@@
 	4350 4950 2250 4950
 Wire Wire Line
-	3450 7400 8600 7400
-Wire Wire Line
-	3450 6750 3450 7400
-Wire Wire Line
-	3400 7450 3400 6200
-Wire Wire Line
-	3400 6200 4050 6200
-Wire Wire Line
-	4050 6200 4050 5650
-Wire Wire Line
-	4050 5650 3700 5650
-Wire Wire Line
-	3400 7450 8550 7450
-Wire Wire Line
 	7850 6900 8900 6900
 Wire Wire Line
@@
 	2500 2750 3200 2750
 Wire Wire Line
-	3900 6300 2050 6300
-Connection ~ 3900 6300
-Wire Wire Line
 	1200 6300 1200 6450
 Wire Wire Line
-	3900 6300 3900 6450
-Wire Wire Line
 	2050 6350 2050 6300
 Connection ~ 2050 6300
@@
 	0    1    1    0
 $EndComp
+$Comp
+L power:GND #PWR051
+U 1 1 6218F136
+P 4500 6900
+F 0 "#PWR051" H 4500 6650 50  0001 C CNN
+F 1 "GND" H 4500 6750 50  0000 C CNN
+F 2 "" H 4500 6900 50  0001 C CNN
+F 3 "" H 4500 6900 50  0001 C CNN
+	1    4500 6900
+	1    0    0    -1
+$EndComp
+Wire Wire Line
+	2050 6300 4450 6300
+Wire Wire Line
+	2350 6950 2500 6950
+Connection ~ 2500 6950
+Wire Wire Line
+	3700 5550 3950 5550
+Wire Wire Line
+	4250 5450 4250 6350
+Wire Wire Line
+	4250 6350 3500 6350
+Wire Wire Line
+	2900 6350 2900 6450
+Connection ~ 4250 5450
+Connection ~ 3500 6350
+Wire Wire Line
+	3500 6350 2900 6350
+$Comp
+L power:GND #PWR050
+U 1 1 624833BA
+P 4150 7150
+F 0 "#PWR050" H 4150 6900 50  0001 C CNN
+F 1 "GND" H 4250 7050 50  0000 C CNN
+F 2 "" H 4150 7150 50  0001 C CNN
+F 3 "" H 4150 7150 50  0001 C CNN
+	1    4150 7150
+	1    0    0    -1
+$EndComp
+$Comp
+L Device:R R13
+U 1 1 6248405A
+P 3500 7000
+F 0 "R13" V 3400 7000 50  0000 C CNN
+F 1 "200" V 3500 7000 50  0000 C CNN
+F 2 "Resistor_SMD:R_1206_3216Metric" V 3430 7000 50  0001 C CNN
+F 3 "~" H 3500 7000 50  0001 C CNN
+	1    3500 7000
+	-1   0    0    1
+$EndComp
+$Comp
+L Device:D_Zener D6
+U 1 1 62484050
+P 3800 7000
+F 0 "D6" H 3800 7200 50  0000 C CNN
+F 1 "MMSZ5231B" H 3800 7100 50  0000 C CNN
+F 2 "Diode_SMD:D_SOD-123F" H 3800 7000 50  0001 C CNN
+F 3 "~" H 3800 7000 50  0001 C CNN
+	1    3800 7000
+	0    1    1    0
+$EndComp
+$Comp
+L Device:R R14
+U 1 1 62484046
+P 4150 7000
+F 0 "R14" V 4050 7000 50  0000 C CNN
+F 1 "400" V 4150 7000 50  0000 C CNN
+F 2 "Resistor_SMD:R_1206_3216Metric" V 4080 7000 50  0001 C CNN
+F 3 "~" H 4150 7000 50  0001 C CNN
+	1    4150 7000
+	-1   0    0    1
+$EndComp
+Wire Wire Line
+	3300 6850 3500 6850
+Wire Wire Line
+	3500 7150 3650 7150
+Wire Wire Line
+	3650 7150 3650 6850
+Wire Wire Line
+	3650 6850 3800 6850
+Wire Wire Line
+	3800 6850 4150 6850
+Connection ~ 3800 6850
+Wire Wire Line
+	4150 6850 4550 6850
+Connection ~ 4150 6850
+Wire Wire Line
+	3800 7150 4150 7150
+Connection ~ 4150 7150
+Wire Wire Line
+	3700 5650 4400 5650
+Wire Wire Line
+	8550 7350 4400 7350
+Wire Wire Line
+	4400 5650 4400 7350
+Wire Wire Line
+	5400 4050 7400 4050
+Wire Wire Line
+	2450 6750 2450 7400
+Wire Wire Line
+	2450 7400 8600 7400
+Connection ~ 2450 6750
 $EndSCHEMATC

Commit message: added BAV99 to analog pins
Parts:
- removed D1, D2, D6: MMSZ5231B, Diode_SMD:D_SOD-123F, symbol Device:D_Zener
- added D1, D2, D6: BAV99, Package_TO_SOT_SMD:SOT-23, symbol Diode:BAV99
- R12: footprint Resistor_SMD:R_1210_3225Metric -> Resistor_SMD:R_1206_3216Metric
- R13, R6, R8: value 200 -> 1K
- R14, R7, R9: value 400 -> 2K
Connections:
- net GND: now also J4.MH1, J4.MH2, R14.2, R9.2, D1.1 (K), D2.1 (K), D6.1 (K); no longer R14.1, R9.1
- net at U6.7 (VIOUT): now also R8.2; no longer R13.2
- net at C1.1, C10.1, C5.1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: now also D1.2 (A), D2.2 (A), D6.2 (A)
- net at J14.2 (Pin_2), R6.1, R7.1: now also D2.3 (K)
- net at R8.1: now also J13.12 (Pin_12), R9.1, D1.3 (K); no longer J6.4
- new net: D6.3 (K), J14.1 (Pin_1), R13.1, R14.1
- new net: J6.4, R13.2
Other:
- moved on the sheet: C4, R6, R7
